File: Blinky/Blinky.kicad_pcb (KiCad board)
At the start: 4 copper layers, 44.7 x 64.6 mm, 97 parts, among them J1 Conn_01x06_Socket, J2 Conn_01x06_Socket, J3 Battery Connector, J4 Charging Notches, J5 Battery Connector, Q1 IRLML6244, Q2 IRLML6244, Q3 IRLML6244, Q4 IRLML6244, Q5 IRLML6244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

Commit message: Kiezburn status
Parts:
- R1, R11: value 4 -> 5.6
- R3, R9: value 1 -> 1.8
- R5, R7: value 1 -> 2
- U4: footprint Library:TSSOP-8_L4.4-W3.0-P0.65-LS6.4-BL-2 -> footprint:SOIC-8_L4.9-W3.9-P1.27-LS6.0-BL
- moved LOGO102 36.0 mm to (172.8, 55.6)
- moved G*** 34.9 mm to (162.3, 53.3)
- moved G*** 4.33 mm to (156.0, 86.4)
- moved U4 1.13 mm to (128.8, 93.0)
- moved J4 0.17 mm to (156.3, 44.5)
- turned R25 to 180 degrees
Connections:
- J2 pad 2: /PIN9 -> /PIN11
- J2 pad 3: /PIN8 -> /PIN16
- U3 pad 11: unconnected-(U3-IO18-Pad11) -> /PIN11
- U3 pad 16: unconnected-(U3-IO46-Pad16) -> /PIN16
- U3 pad 32: /32_32khz -> unconnected-(U3-IO39-Pad32)
- U3 pad 33: /33_32khz -> unconnected-(U3-IO40-Pad33)
- U3 pad 8: /PIN8 -> /32_32khz
- U3 pad 9: /PIN9 -> /33_32khz
Routing:
- net /PIN16: track 0.00 -> 37.1 mm, vias 0 -> 2
- net /PIN11: track 0.00 -> 33.3 mm, vias 0 -> 2
- net /PIN9: track 32.8 -> 0.00 mm, vias 2 -> 0
- net /PIN8: track 31.4 -> 0.00 mm, vias 2 -> 0
- net VDD: track 21.7 -> 31.9 mm, vias 10 -> 9
- net /32_32khz: track 15.8 -> 23.2 mm
- net Net-(U4A-IN1-): track 8.37 -> 10.4 mm, vias 2 -> 1
- net GND: track 92.6 -> 91.5 mm
- net /VDD_REF: track 18.5 -> 19.6 mm
- net Net-(U4B-IN2-): track 17.1 -> 17.9 mm
- net /33_32khz: track 19.4 -> 18.6 mm
- net /BLUE1: track 64.8 -> 65.3 mm
