File: Blinky/Blinky.kicad_sch (KiCad schematic)
At the start: 79 parts, among them J1 Conn_01x06_Socket, J2 Conn_01x06_Socket, J3 Battery Connector, J4 Charging Notches, J5 Battery Connector, Q1 IRLML6244, Q2 IRLML6244, Q3 IRLML6244, Q4 IRLML6244, Q5 IRLML6244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

Commit message: Kiezburn status
Parts:
- J3, J5: footprint Connector_JST:JST_PH_B2B-PH-K_1x02_P2.00mm_Vertical -> footprint:CONN-TH_S2B-PH-K-LF-SN
- R1, R11: value 4 -> 5.6
- R3, R9: value 1 -> 1.8
- R5, R7: value 1 -> 2
- U4: footprint Library:TSSOP-8_L4.4-W3.0-P0.65-LS6.4-BL-2 -> footprint:SOIC-8_L4.9-W3.9-P1.27-LS6.0-BL
Connections:
- net 32_32khz: now also U3.8 (IO15); no longer U3.32 (IO39)
- net 33_32khz: now also U3.9 (IO16); no longer U3.33 (IO40)
- net PIN11: now reaches U3.11 (IO18)
- net PIN11: now also J2.2 (Pin_2)
- net PIN16: now reaches U3.16 (IO46)
- net PIN16: now also J2.3 (Pin_3)
- removed net PIN8: J2.3 (Pin_3), U3.8 (IO15)
- removed net PIN9: J2.2 (Pin_2), U3.9 (IO16)
Changed lines of the file:
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@@
 	(wire
 		(pts
+			(xy 180.34 149.86) (xy 189.23 149.86)
+		)
+		(stroke
+			(width 0)
+			(type default)
+		)
+	)
+	(wire
+		(pts
 			(xy 367.03 62.23) (xy 374.65 62.23)
 		)
@@
 	(wire
 		(pts
+			(xy 180.34 137.16) (xy 189.23 137.16)
+		)
+		(stroke
+			(width 0)
+			(type default)
+		)
+	)
+	(wire
+		(pts
 			(xy 302.26 44.45) (xy 302.26 48.26)
 		)
@@
 		)
 	)
+	(label "33_32khz"
+		(at 180.34 132.08 0)
+		(fields_autoplaced yes)
+		(effects
+			(font
+				(size 1.27 1.27)
+			)
+			(justify left bottom)
+		)
+	)
 	(label "VDD_REF"
 		(at 322.58 199.39 0)
@@
 		)
 	)
-	(label "PIN8"
-		(at 181.61 129.54 0)
-		(fields_autoplaced yes)
-		(effects
-			(font
-				(size 1.27 1.27)
-			)
-			(justify left bottom)
-		)
-	)
-	(label "33_32khz"
-		(at 213.36 129.54 0)
-		(fields_autoplaced yes)
-		(effects
-			(font
-				(size 1.27 1.27)
-			)
-			(justify left bottom)
-		)
-	)
 	(label "BAT+"
 		(at 353.06 38.1 0)
@@
 		)
 	)
-	(label "PIN9"
-		(at 181.61 132.08 0)
+	(label "PIN11"
+		(at 181.61 137.16 0)
 		(fields_autoplaced yes)
 		(effects
@@
 		)
 	)
+	(label "32_32khz"
+		(at 180.34 129.54 0)
+		(fields_autoplaced yes)
+		(effects
+			(font
+				(size 1.27 1.27)
+			)
+			(justify left bottom)
+		)
+	)
 	(label "PIN7"
 		(at 181.61 127 0)
@@
 		)
 	)
-	(label "PIN8"
+	(label "PIN16"
 		(at 247.65 100.33 0)
 		(fields_autoplaced yes)
@@
 		)
 	)
-	(label "PIN9"
+	(label "PIN11"
 		(at 247.65 102.87 0)
 		(fields_autoplaced yes)
@@
 		)
 	)
-	(label "BAT+"
-		(at 381 101.6 0)
+	(label "PIN16"
+		(at 181.61 149.86 0)
 		(fields_autoplaced yes)
 		(effects
@@
 		)
 	)
-	(label "32_32khz"
-		(at 213.36 132.08 0)
+	(label "BAT+"
+		(at 381 101.6 0)
 		(fields_autoplaced yes)
 		(effects
@@
 			)
 		)
-		(property "Value" "1"
+		(property "Value" "2"
 			(at 102.87 167.64 0)
 			(effects
@@
 			)
 		)
-		(property "Value" "4"
+		(property "Value" "5.6"
 			(at 100.33 200.66 0)
 			(effects
@@
 			)
 		)
-		(property "Value" "4"
+		(property "Value" "5.6"
 			(at 104.14 147.32 0)
 			(effects
@@
 			)
 		)
-		(property "Value" "1"
+		(property "Value" "1.8"
 			(at 101.6 184.15 0)
 			(effects
@@
 			)
 		)
-		(property "Footprint" "Connector_JST:JST_PH_B2B-PH-K_1x02_P2.00mm_Vertical"
+		(property "Footprint" "footprint:CONN-TH_S2B-PH-K-LF-SN"
 			(at 377.19 30.48 0)
 			(effects
@@
 			)
 		)
-		(property "Footprint" "Connector_JST:JST_PH_B2B-PH-K_1x02_P2.00mm_Vertical"
+		(property "Footprint" "footprint:CONN-TH_S2B-PH-K-LF-SN"
 			(at 377.19 38.1 0)
 			(effects
@@
 			)
 		)
-		(property "Value" "1"
+		(property "Value" "2"
 			(at 104.14 114.3 0)
 			(effects
@@
 			)
 		)
-		(property "Footprint" "Library:TSSOP-8_L4.4-W3.0-P0.65-LS6.4-BL-2"
+		(property "Footprint" "footprint:SOIC-8_L4.9-W3.9-P1.27-LS6.0-BL"
 			(at 311.15 191.77 0)
 			(effects
@@
 			)
 		)
-		(property "Value" "1"
+		(property "Value" "1.8"
 			(at 104.14 130.81 0)
 			(effects
@@
 			)
 		)
-		(property "Footprint" "Library:TSSOP-8_L4.4-W3.0-P0.65-LS6.4-BL-2"
+		(property "Footprint" "footprint:SOIC-8_L4.9-W3.9-P1.27-LS6.0-BL"
 			(at 276.86 191.77 0)
 			(effects
